Commit message: Updated the MP-400 with the correct laser scanner topics

File: robots/mp_400/mp_400.urdf (robot description, URDF)
Before this commit: robot mp_400, 9 links, 8 joints
Links:
- removed link laser_1_link
- added link lidar_1_link, mass 0.001; collision mesh filename=package://neo_simulation2/robots/mp_400/meshes/SICK-MICROSC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 scale=0.001 0.001 0.001; visual mesh filename=package://neo_simulation2/robots/mp_400/meshes/SICK-MICROSC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 scale=0.001 0.001 0.001
Joints:
- joint laser_1_joint: child laser_1_link -> lidar_1_link

Commit message: cleanup2: Files Restructuring

File: robots/mp_400/mp_400.urdf (robot description, URDF)
Before this commit: robot mp_400, 9 links, 8 joints
Links:
- link lidar_1_link: geometry collision mesh filename=package://neo_simulation2/components/sensors/SICK-MICROSCAN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 scale=0.001 0.001 0.001; visual mesh filename=package://neo_simulation2/components/sensors/SICK-MICROSCAN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 scale=0.001 0.001 0.001

File: robots/mp_500/mp_500.urdf (robot description, URDF)
Before this commit: robot mp_500, 6 links, 5 joints
Links:
- link lidar_1_link: geometry collision mesh filename=package://neo_simulation2/components/sensors/SICK-S300.dae scale=0.001 0.001 0.001; visual mesh filename=package://neo_simulation2/components/sensors/SICK-S300.dae scale=0.001 0.001 0.001

File: robots/mpo_500/mpo_500.urdf (robot description, URDF)
Before this commit: robot mpo_500, 8 links, 7 joints
Links:
- link lidar_1_link: geometry collision mesh filename=package://neo_simulation2/components/sensors/SICK-MICROSCAN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 scale=0.001 0.001 0.001; visual mesh filename=package://neo_simulation2/components/sensors/SICK-MICROSCAN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 scale=0.001 0.001 0.001
- link lidar_2_link: geometry collision mesh filename=package://neo_simulation2/components/sensors/SICK-MICROSCAN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 scale=0.001 0.001 0.001; visual mesh filename=package://neo_simulation2/components/sensors/SICK-MICROSCAN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 scale=0.001 0.001 0.001

File: robots/mpo_700/mpo_700.urdf (robot description, URDF)
Before this commit: robot mpo_700, 12 links, 11 joints
Links:
- link lidar_1_link: geometry collision mesh filename=package://neo_simulation2/components/sensors/SICK-S300.dae scale=0.001 0.001 0.001; visual mesh filename=package://neo_simulation2/components/sensors/SICK-S300.dae scale=0.001 0.001 0.001
- link lidar_2_link: geometry collision mesh filename=package://neo_simulation2/components/sensors/SICK-S300.dae scale=0.001 0.001 0.001; visual mesh filename=package://neo_simulation2/components/sensors/SICK-S300.dae scale=0.001 0.001 0.001
