Commit message: adding EC 66 with mpo-700

File: robots/mpo_700/mpo_700.urdf.xacro (robot description, xacro)
@@ -4,9 +4,9 @@
 <!-- |    EDITING THIS FILE BY HAND IS NOT RECOMMENDED                                 | -->
 <!-- =================================================================================== -->
-<robot name="mpo_700">
+<robot xmlns:xacro="http://www.ros.org/wiki/xacro" name="mpo_700">
   <!-- SENSORS -->
   <!-- Sick S300 - Comment/Uncomment if required -->
-  <!-- <xacro:include filename="$(find neo_simulation2)/robots/mpo_700/xacros/sick_S300.xacro" /> -->
   <!--Ultrasonics, cameras and IMU's  -->
+<xacro:arg name="include_arm" default="false"/>
   <gazebo reference="lidar_1_link">
     <sensor name="lidar_1_sensor" type="ray">
@@ -454,43 +454,329 @@
     <mu2>0.0001</mu2>
   </gazebo>
-<!-- <joint name="camera_joint" type="fixed">
-    <axis xyz="0 1 0"/>
-    <origin rpy="0 0 3.14159" xyz="-0.228 0.015 0.461"/>
-    <parent link="base_link"/>
-    <child link="camera_link"/>
-  </joint>
-  <joint name="camera_optical_joint" type="fixed">
-    <origin rpy="-1.5707963267948966 0 -1.5707963267948966" xyz="0 0.015 0"/>
-    <parent link="camera_link"/>
-    <child link="camera_link_optical"/>
-  </joint>
-  <joint name="camera_gazebo_joint" type="fixed">
-    <origin rpy="0 0 0" xyz="0 0.015 0"/>
-    <parent link="camera_link"/>
-    <child link="camera_link_gazebo"/>
-  </joint>
-  <link name="camera_link">
-    <collision>
-      <origin rpy="0 0 0" xyz="0 0 0"/>
-      <geometry>
-        <box size="0.05 0.05 0.05"/>
-      </geometry>
-    </collision>
-    <visual>
-      <origin rpy="1.570796 0 1.570796" xyz="0 -0.0175 0"/>
-      <geometry>
-        <mesh filename="package://neo_simulation2/components/sensors/d435.dae"/>
-      </geometry>
-      <material name="red">
-        <color rgba="1 0 0 1"/>
-      </material>
-    </visual>
-    <inertial>
-      <mass value="1e-5"/>
-      <origin rpy="0 0 0" xyz="0 0 0"/>
-      <inertia ixx="1e-6" ixy="0" ixz="0" iyy="1e-6" iyz="0" izz="1e-6"/>
-    </inertial>
-  </link>
-  <link name="camera_link_optical"/>
-  <link name="camera_link_gazebo"/> -->
+  <!--cabinet-->
+  <joint name="cabinet_joint" type="fixed">
+    <parent link="base_link" />
+    <child link="cabinet_link" />
+    <origin xyz="0.072 0 0.35" rpy="0 0 0" />
+   </joint>
+    <link name="cabinet_link">
+      <inertial>
+        <mass value="2" />
+        <origin xyz="0 0 0" rpy="0 0 0"/>
+        <inertia ixx="0.457072" ixy="0.0" ixz="0.0"
+                 iyy="0.23616" iyz="0.0"
+                 izz="0.686" />
+      </inertial>
+      <visual>
+        <origin xyz="0 0 0" rpy="0 0 -1.5708" />
+        <geometry>
+            <mesh filename="package://neo_simulation2/components/arms/cabinet.dae" scale="0.001 0.001 0.001"/>
+        </geometry>
+      </visual>
+      <collision>
+        <origin xyz="0 0 0" rpy="0 0 -1.5708" />
+        <geometry>
+            <mesh filename="package://neo_simulation2/components/arms/cabinet.dae" scale="0.001 0.001 0.001"/>
+        </geometry>
+      </collision>
+    </link>
+  <!-- EC 66 -->
+    <joint name="arm_joint" type="fixed">
+        <origin xyz="0.133 0.0 0.485" rpy="0.0 0.0 0.0" />
+        <parent link="cabinet_link" />
+        <child link="arm_base_link" />
+    </joint>
+    <link name="arm_base_link">
+        <inertial>
+            <origin xyz="0.00039768 8.0247E-10 0.012605" rpy="0 0 0" />
+            <mass value="0.41542" />
+            <inertia ixx="0.00054632" ixy="-4.5067E-09" ixz="5.9528E-07" iyy="0.00053741" iyz="-3.5275E-10" izz="0.0010336" />
+        </inertial>
+        <visual>
+            <origin xyz="0 0 0" rpy="0 0 0" />
+            <geometry>
+                <mesh filename="package://neo_simulation2/components/arms/ec66/meshes/base_link.stl" />
+            </geometry>
+        </visual>
+        <collision>
+            <origin xyz="0 0 0" rpy="0 0 0" />
+            <geometry>
+                <mesh filename="package://neo_simulation2/components/arms/ec66/meshes/base_link.stl" />
+            </geometry>
+        </collision>
+    </link>
+    <link name="link1">
+        <inertial>
+            <origin xyz="3.9336E-06 -0.0082614 0.0028405" rpy="0 0 0" />
+            <mass value="1.7827" />
+            <inertia ixx="0.0031691" ixy="-1.2175E-07" ixz="-2.8349E-08" iyy="0.0029334" iyz="0.00037927" izz="0.0035086" />
+        </inertial>
+        <visual>
+            <origin xyz="0 0 0" rpy="0 0 0" />
+            <geometry>
+                <mesh filename="package://neo_simulation2/components/arms/ec66/meshes/link1.stl" />
+            </geometry>
+            <material name="">
+                <color rgba="1 1 1 1" />
+            </material>
+        </visual>
+        <collision>
+            <origin xyz="0 0 0" rpy="0 0 0" />
+            <geometry>
+                <mesh filename="package://neo_simulation2/components/arms/ec66/meshes/link1.stl" />
+            </geometry>
+        </collision>
+    </link>
+    <joint name="joint1" type="revolute">
+        <parent link="arm_base_link" />
+        <child link="link1" />
+        <axis xyz="0 0 1" />
+        <limit lower="-6.2832" upper="6.2832" effort="150.0" velocity="2.61993" />
+        <dynamics damping="1.5" friction="3.5" />
+    </joint>
+    <link name="link2">
+        <inertial>
+            <origin xyz="-2.17E-06 0.17637 0.13932" rpy="0 0 0" />
+            <mass value="4.8843" />
+            <inertia ixx="0.022101" ixy="-1.0832E-07" ixz="-1.2727E-07" iyy="0.0066105" iyz="-0.00021178" izz="0.022526" />
+        </inertial>
+        <visual>
+            <origin xyz="0 0 0" rpy="0 0 0" />
+            <geometry>
+                <mesh filename="package://neo_simulation2/components/arms/ec66/meshes/link2.stl" />
+            </geometry>
+            <material name="">
+                <color rgba="1 1 1 1" />
+            </material>
+        </visual>
+        <collision>
+            <origin xyz="0 0 0" rpy="0 0 0" />
+            <geometry>
+                <mesh filename="package://neo_simulation2/components/arms/ec66/meshes/link2.stl" />
+            </geometry>
+        </collision>
+    </link>
+    <joint name="joint2" type="revolute">
+        <origin xyz="0 0 0" rpy="1.5708 -1.5708 0" />
+        <parent link="link1" />
+        <child link="link2" />
+        <axis xyz="0 0 1" />
+        <limit lower="-3.14" upper="0" effort="150.0" velocity="2.61993" />
+        <dynamics damping="1.5" friction="3.5" />
+    </joint>
+    <link name="link3">
+        <inertial>
+            <origin xyz="0.20069 -7.9845E-06 0.028008" rpy="0 0 0" />
+            <mass value="2.1495" />
+            <inertia ixx="0.0015747" ixy="-2.8912E-08" ixz="7.3471E-05" iyy="0.0091566" iyz="-1.4815E-07" izz="0.0091573" />
+        </inertial>
+        <visual>
+            <origin xyz="0 0 0" rpy="0 0 0" />
+            <geometry>
+                <mesh filename="package://neo_simulation2/components/arms/ec66/meshes/link3.stl" />
+            </geometry>
+            <material name="">
+                <color rgba="1 1 1 1" />
+            </material>
+        </visual>
+        <collision>
+            <origin xyz="0 0 0" rpy="0 0 0" />
+            <geometry>
+                <mesh filename="package://neo_simulation2/components/arms/ec66/meshes/link3.stl" />
+            </geometry>
+        </collision>
+    </link>
+    <joint name="joint3" type="revolute">
+        <origin xyz="0 0.418 0" rpy="0 0 1.10" />
+        <parent link="link2" />
+        <child link="link3" />
+        <axis xyz="0 0 1" />
+        <limit lower="-2.7925" upper="2.7925" effort="150.0" velocity="3.31613" />
+        <dynamics damping="1.5" friction="3.5" />
+    </joint>
+    <link name="link4">
+        <inertial>
+            <origin xyz="-5.2274E-07 -0.00070291 -0.006006" rpy="0 0 0" />
+            <mass value="0.53436" />
+            <inertia ixx="0.00041486" ixy="-4.7177E-09" ixz="-1.1841E-09" iyy="0.0004403" iyz="-5.8283E-05" izz="0.00037669" />
+        </inertial>
+        <visual>
+            <origin xyz="0 0 0" rpy="0 0 0" />
+            <geometry>
+                <mesh filename="package://neo_simulation2/components/arms/ec66/meshes/link4.stl" />
+            </geometry>
+            <material name="">
+                <color rgba="1 1 1 1" />
+            </material>
+        </visual>
+        <collision>
+            <origin xyz="0 0 0" rpy="0 0 0" />
+            <geometry>
+                <mesh filename="package://neo_simulation2/components/arms/ec66/meshes/link4.stl" />
+            </geometry>
+        </collision>
+    </link>
+    <joint name="joint4" type="revolute">
+        <origin xyz="0.398 0 0.122" rpy="0 0 0" />
+        <parent link="link3" />
+        <child link="link4" />
+        <axis xyz="0 0 1" />
+        <limit lower="-6.2832" upper="6.2832" effort="28.0" velocity="4.53786" />
+        <dynamics damping="1.5" friction="3.5" />
+    </joint>
+    <link name="link5">
+        <inertial>
+            <origin xyz="5.2283E-07 0.00070291 -0.006006" rpy="0 0 0" />
+            <mass value="0.53436" />
+            <inertia ixx="0.00041486" ixy="-4.6787E-09" ixz="1.1524E-09" iyy="0.0004403" iyz="5.8283E-05" izz="0.00037669" />
+        </inertial>
+        <visual>
+            <origin xyz="0 0 0" rpy="0 0 0" />
+            <geometry>
+                <mesh filename="package://neo_simulation2/components/arms/ec66/meshes/link5.stl" />
+            </geometry>
+            <material name="">
+                <color rgba="1 1 1 1" />
+            </material>
+        </visual>
+        <collision>
+            <origin xyz="0 0 0" rpy="0 0 0" />
+            <geometry>
+                <mesh filename="package://neo_simulation2/components/arms/ec66/meshes/link5.stl" />
+            </geometry>
+        </collision>
+    </link>
+    <joint name="joint5" type="revolute">
+        <origin xyz="0 0.098 0" rpy="1.5708 0 -3.1416" />
+        <parent link="link4" />
+        <child link="link5" />
+        <axis xyz="0 0 1" />
+        <limit lower="-6.2832" upper="6.2832" effort="28.0" velocity="4.53786" />
+        <dynamics damping="1.5" friction="3.5" />
+    </joint>
+    <link name="link6">
+        <inertial>
+            <origin xyz="-1.7556E-08 -0.00045052 -0.021169" rpy="0 0 0" />
+            <mass value="0.16488" />
+            <inertia ixx="7.7869E-05" ixy="-3.3531E-10" ixz="1.915E-10" iyy="7.757E-05" iyz="-7.8331E-08" izz="0.00011744" />
+        </inertial>
+        <visual>
+            <origin xyz="0 0 0" rpy="0 0 0" />
+            <geometry>
+                <mesh filename="package://neo_simulation2/components/arms/ec66/meshes/link6.stl" />
+            </geometry>
+            <material name="">
+                <color rgba="0.79216 0.81961 0.93333 1" />
+            </material>
+        </visual>
+        <collision>
+            <origin xyz="0 0 0" rpy="0 0 0" />
+            <geometry>
+                <mesh filename="package://neo_simulation2/components/arms/ec66/meshes/link6.stl" />
+            </geometry>
+        </collision>
+    </link>
+    <joint name="joint6" type="revolute">
+        <origin xyz="0 -0.089 0" rpy="-1.5708 0 3.1416" />
+        <parent link="link5" />
+        <child link="link6" />
+        <axis xyz="0 0 1" />
+        <limit lower="-6.2832" upper="6.2832" effort="28.0" velocity="4.53786" />
+        <dynamics damping="1.5" friction="3.5" />
+    </joint>
+    <link name="flan" />
+    <joint name="flan_joint" type="fixed">
+        <origin xyz="0 0 0" rpy="0 0 0" />
+        <parent link="link6" />
+        <child link="flan" />
+    </joint>
+    <ros2_control name="GazeboSystem" type="system">
+        <hardware>
+            <plugin>gazebo_ros2_control/GazeboSystem</plugin>
+               <parameters>$(find neo_simulation2)/configs/arms/joint_names_ec66_description.yaml</parameters>
+            </hardware>
+        <joint name="joint1">
+            <command_interface name="position">
+                <param name="min">-3.15</param>
+                <param name="max">3.15</param>
+            </command_interface>
+            <command_interface name="velocity">
+                <param name="min">-3.15</param>
+                <param name="max">3.15</param>
+            </command_interface>
+            <state_interface name="position"/>
+            <state_interface name="velocity"/>
+            <state_interface name="effort"/>
+        </joint>
+        <joint name="joint2">
+            <command_interface name="position">
+                <param name="min">-3.15</param>
+                <param name="max">3.15</param>
+            </command_interface>
+            <command_interface name="velocity">
+                <param name="min">-3.15</param>
+                <param name="max">3.15</param>
+            </command_interface>
+            <state_interface name="position"/>
+            <state_interface name="velocity"/>
+            <state_interface name="effort"/>
+        </joint>
+        <joint name="joint3">
+            <command_interface name="position">
+                <param name="min">-3.15</param>
+                <param name="max">3.15</param>
+            </command_interface>
+            <command_interface name="velocity">
+                <param name="min">-3.15</param>
+                <param name="max">3.15</param>
+            </command_interface>
+            <state_interface name="position"/>
+            <state_interface name="velocity"/>
+            <state_interface name="effort"/>
+        </joint>
+        <joint name="joint4">
+            <command_interface name="position">
+                <param name="min">-3.15</param>
+                <param name="max">3.15</param>
+            </command_interface>
+            <command_interface name="velocity">
+                <param name="min">-3.15</param>
+                <param name="max">3.15</param>
+            </command_interface>
+            <state_interface name="position"/>
+            <state_interface name="velocity"/>
+            <state_interface name="effort"/>
+        </joint>
+        <joint name="joint5">
+            <command_interface name="position">
+                <param name="min">-3.15</param>
+                <param name="max">3.15</param>
+            </command_interface>
+            <command_interface name="velocity">
+                <param name="min">-3.15</param>
+                <param name="max">3.15</param>
+            </command_interface>
+            <state_interface name="position"/>
+            <state_interface name="velocity"/>
+            <state_interface name="effort"/>
+        </joint>
+        <joint name="joint6">
+            <command_interface name="position">
+                <param name="min">-3.15</param>
+                <param name="max">3.15</param>
+            </command_interface>
+            <command_interface name="velocity">
+                <param name="min">-3.15</param>
+                <param name="max">3.15</param>
+            </command_interface>
+            <state_interface name="position"/>
+            <state_interface name="velocity"/>
+            <state_interface name="effort"/>
+        </joint>
+    </ros2_control>
+    <gazebo>
+        <plugin filename="libgazebo_ros2_control.so" name="gazebo_ros2_control">
+           <parameters> /home/youknowwho/neobotix_workspace/src/elite_description/config/joint_names_ec66_description.yaml </parameters>
+        </plugin>
+    </gazebo>
 </robot>

Commit message: adding UR10

File: robots/mpo_700/mpo_700.urdf.xacro (robot description, xacro)
@@ -8,5 +8,6 @@
   <!-- Sick S300 - Comment/Uncomment if required -->
   <!--Ultrasonics, cameras and IMU's  -->
-<xacro:arg name="include_arm" default="false"/>
+<xacro:arg name="ur10" default="false"/>
+<xacro:arg name="elite" default="false"/>
   <gazebo reference="lidar_1_link">
     <sensor name="lidar_1_sensor" type="ray">
@@ -455,13 +456,29 @@
   </gazebo>
   <!--cabinet-->
-<xacro:if value="$(arg include_arm)">
+<xacro:if value="$(arg ur10)">
   <xacro:include filename="$(find neo_simulation2)/components/arms/cabinet.urdf.xacro" />
-  <xacro:include filename="$(find neo_simulation2)/components/arms/ec66/ec66_description.urdf.xacro" />
   <!-- cabinet -->
   <xacro:cabinet name="cabinet" parent="base_link">
     <origin xyz="0.072 0 0.35" rpy="0 0 0" />
   </xacro:cabinet>
-  <xacro:ec66 name="ec_66" parent="cabinet_link">
-    <origin xyz="0.133 0.0 0.485" rpy="0.0 0.0 0.0" />
+  <xacro:include filename="$(find neo_simulation2)/components/arms/ur10/ur10.urdf.xacro" />
+  <xacro:ur10_robot parent="cabinet_link" prefix="ur10" joint_limited="true"
+     shoulder_pan_lower_limit="${-pi}" shoulder_pan_upper_limit="${pi}"
+     shoulder_lift_lower_limit="${-pi}" shoulder_lift_upper_limit="${pi}"
+     elbow_joint_lower_limit="${-pi}" elbow_joint_upper_limit="${pi}"
+     wrist_1_lower_limit="${-pi}" wrist_1_upper_limit="${pi}"
+     wrist_2_lower_limit="${-pi}" wrist_2_upper_limit="${pi}"
+     wrist_3_lower_limit="${-pi}" wrist_3_upper_limit="${pi}">
+  </xacro:ur10_robot>
+</xacro:if>
+<xacro:if value="$(arg elite)">
+  <xacro:include filename="$(find neo_simulation2)/components/arms/cabinet.urdf.xacro" />
+  <!-- cabinet -->
+  <xacro:cabinet name="cabinet" parent="base_link">
+    <origin xyz="0.072 0 0.35" rpy="0 0 0" />
+  </xacro:cabinet>
+  <xacro:include filename="$(find neo_simulation2)/components/arms/ec66/ec66_description.urdf.xacro" />
+    <xacro:ec66 name="ec_66" parent="cabinet_link">
+      <origin xyz="0.133 0.0 0.485" rpy="0.0 0.0 0.0" />
   </xacro:ec66>
 </xacro:if>
