Commit message: Navigation stack initial set up for MPO-700

File: robots/mpo_700/mpo_700.urdf (robot description, URDF)
Before this commit: robot mpo_700, 13 links, 12 joints
Joints:
- joint base_footprint_joint: origin xyz=0.24 0.18 0.22 rpy=0 0 3.14 -> xyz=0 0 0 rpy=0 0 3.14

Commit message: Added friction components to MPO-700 robot model-makes it smoother

File: robots/mpo_700/mpo_700.urdf (robot description, URDF)
Before this commit: robot mpo_700, 13 links, 12 joints
Links:
- removed link docking_adapter_link
- link lidar_1_link: mass 0.0001 -> 1.2; geometry collision mesh filename=package://neo_simulation2/robots/mpo_700/meshes/SICK-S300.d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 scale=0.001 0.001 0.001; visual mesh filename=package://neo_simulation2/robots/mpo_700/meshes/SICK-S300.d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 scale=0.001 0.001 0.001
- link lidar_2_link: mass 0.0001 -> 0.001; geometry collision mesh filename=package://neo_simulation2/robots/mpo_700/meshes/SICK-S300.d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 scale=0.001 0.001 0.001; visual mesh filename=package://neo_simulation2/robots/mpo_700/meshes/SICK-S300.d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 scale=0.001 0.001 0.001
- link mpo_700_wheel_back_left_link: geometry collision mesh filename=package://neo_simulation2/robots/mpo_700/meshes/MPO-700-WHE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 scale=0.001 0.001 0.001; visual mesh filename=package://neo_simulation2/robots/mpo_700/meshes/MPO-700-WHE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 scale=0.001 0.001 0.001
- link mpo_700_wheel_back_right_link: geometry collision mesh filename=package://neo_simulation2/robots/mpo_700/meshes/MPO-700-WHE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 scale=0.001 0.001 0.001; visual mesh filename=package://neo_simulation2/robots/mpo_700/meshes/MPO-700-WHE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 scale=0.001 0.001 0.001
- link mpo_700_wheel_front_left_link: mass 1.2 -> 2; geometry collision mesh filename=package://neo_simulation2/robots/mpo_700/meshes/MPO-700-WHE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 scale=0.001 0.001 0.001; visual mesh filename=package://neo_simulation2/robots/mpo_700/meshes/MPO-700-WHE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 scale=0.001 0.001 0.001
- link mpo_700_wheel_front_right_link: geometry collision mesh filename=package://neo_simulation2/robots/mpo_700/meshes/MPO-700-WHE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 scale=0.001 0.001 0.001; visual mesh filename=package://neo_simulation2/robots/mpo_700/meshes/MPO-700-WHE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 scale=0.001 0.001 0.001
Joints:
- removed joint docking_adapter_joint
- joint base_footprint_joint: axis 0 0 1 -> 0 0 -1; limit lower=-1e+16 upper=1e+16 effort=1000.0 velocity=6.5 -> (none); origin xyz=0 0 0 rpy=0 0 3.14 -> xyz=0 0 0 rpy=0 0 0
- joint mpo_700_caster_back_left_joint: axis 0 0 1 -> 0 0 -1; limit lower=-1e+16 upper=1e+16 effort=1000.0 velocity=6.5 -> (none); origin xyz=-0.24 0.18 0.22 rpy=0 0 3.14 -> xyz=0.24 -0.18 0.27 rpy=3.14 0 1.57
- joint mpo_700_caster_back_right_joint: axis 0 0 1 -> 0 0 -1; limit lower=-1e+16 upper=1e+16 effort=1000.0 velocity=6.5 -> (none); origin xyz=-0.24 -0.18 0.22 rpy=0 0 0 -> xyz=-0.24 0.18 0.27 rpy=3.14 0 -1.57
- joint mpo_700_caster_front_left_joint: axis 0 0 1 -> 0 0 -1; limit lower=-1e+16 upper=1e+16 effort=1000.0 velocity=6.5 -> (none); origin xyz=0.24 0.18 0.22 rpy=0 0 3.14 -> xyz=0.24 0.18 0.27 rpy=3.14 0 -1.57
- joint mpo_700_caster_front_right_joint: axis 0 0 1 -> 0 0 -1; limit lower=-1e+16 upper=1e+16 effort=1000.0 velocity=6.5 -> (none); origin xyz=0.24 -0.18 0.22 rpy=0 0 0 -> xyz=-0.24 -0.18 0.27 rpy=3.14 0 1.57
- joint mpo_700_wheel_back_left_joint: axis 0 -1 0 -> 1 0 0; limit lower=-1e+16 upper=1e+16 effort=1000.0 velocity=20.5 -> (none); origin xyz=0.0 0.045 -0.12 rpy=0 0 0 -> xyz=-0.05 0. 0.18 rpy=0 0 0
- joint mpo_700_wheel_back_right_joint: axis 0 -1 0 -> 1 0 0; limit lower=-1e+16 upper=1e+16 effort=1000.0 velocity=20.5 -> (none); origin xyz=0.0 -0.045 -0.12 rpy=0 0 3.14 -> xyz=-0.05 0. 0.18 rpy=0 0 0
- joint mpo_700_wheel_front_left_joint: axis 0 -1 0 -> 1 0 0; limit lower=-1e+16 upper=1e+16 effort=1000.0 velocity=20.5 -> lower=-1e+16 upper=1e+16 effort=1000.0 velocity=15; origin xyz=0.0 0.045 -0.12 rpy=0 0 0 -> xyz=-0.05 0. 0.18 rpy=0 0 0
- joint mpo_700_wheel_front_right_joint: axis 0 -1 0 -> 1 0 0; limit lower=-1e+16 upper=1e+16 effort=1000.0 velocity=20.5 -> lower=-1e+16 upper=1e+16 effort=1000.0 velocity=15; origin xyz=0.0 -0.045 -0.12 rpy=0 0 3.14 -> xyz=-0.05 0. 0.18 rpy=0 0 0

Commit message: initia commit that loads the gazebo controllers

File: robots/mpo_700/mpo_700.urdf (robot description, URDF)
Before this commit: robot mpo_700, 15 links, 14 joints
Joints:
- joint mpo_700_caster_back_left_joint: limit (none) -> lower=-1e+16 upper=1e+16 effort=1000.0 velocity=15; type fixed -> revolute
- joint mpo_700_caster_back_right_joint: limit (none) -> lower=-1e+16 upper=1e+16 effort=1000.0 velocity=15; type fixed -> revolute
- joint mpo_700_caster_front_left_joint: limit (none) -> lower=-1e+16 upper=1e+16 effort=1000.0 velocity=15; type fixed -> revolute
- joint mpo_700_caster_front_right_joint: limit (none) -> lower=-1e+16 upper=1e+16 effort=1000.0 velocity=15; type fixed -> revolute
- joint mpo_700_wheel_back_left_joint: limit (none) -> lower=-1e+16 upper=1e+16 effort=1000.0 velocity=15; type fixed -> revolute
- joint mpo_700_wheel_back_right_joint: limit (none) -> lower=-1e+16 upper=1e+16 effort=1000.0 velocity=15; type fixed -> revolute
- joint mpo_700_wheel_front_left_joint: type fixed -> revolute
- joint mpo_700_wheel_front_right_joint: type fixed -> revolute

Commit message: removing the overhead by removing the camera data

File: robots/mpo_700/mpo_700.urdf (robot description, URDF)
Before this commit: robot mpo_700, 15 links, 14 joints
Links:
- removed link camera_link
- removed link camera_link_gazebo
- removed link camera_link_optical
Joints:
- removed joint camera_gazebo_joint
- removed joint camera_joint
- removed joint camera_optical_joint

Commit message: updating the world and the models

File: robots/mpo_700/mpo_700.urdf (robot description, URDF)
Before this commit: robot mpo_700, 12 links, 11 joints
Links:
- link mpo_700_wheel_back_left_link: geometry collision sphere radius=0.09; visual mesh filename=package://neo_simulation2/robots/mpo_700/meshes/MPO-700-WHE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 scale=0.001 0.001 0.001
- link mpo_700_wheel_back_right_link: geometry collision sphere radius=0.09; visual mesh filename=package://neo_simulation2/robots/mpo_700/meshes/MPO-700-WHE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 scale=0.001 0.001 0.001
- link mpo_700_wheel_front_left_link: geometry collision sphere radius=0.09; visual mesh filename=package://neo_simulation2/robots/mpo_700/meshes/MPO-700-WHE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 scale=0.001 0.001 0.001
- link mpo_700_wheel_front_right_link: geometry collision sphere radius=0.09; visual mesh filename=package://neo_simulation2/robots/mpo_700/meshes/MPO-700-WHE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 scale=0.001 0.001 0.001
