Commit message: updates to moveit configs

File: components/arms/ur10/ur10.urdf.xacro (robot description, xacro)
@@ -73,7 +73,7 @@
       </xacro:cylinder_inertial>
     </link>
-    <joint name="shoulder_pan_joint" type="revolute">
+    <joint name="ur10shoulder_pan_joint" type="revolute">
       <parent link="ur10_base_link" />
-      <child link = "shoulder_link" />
+      <child link = "ur10shoulder_link" />
       <origin xyz="0.0 0.0 ${shoulder_height}" rpy="0.0 0.0 0.0" />
       <axis xyz="0 0 1" />
@@ -86,5 +86,5 @@
       <dynamics damping="0.5" friction="10.0"/>
     </joint>
-    <link name="shoulder_link">
+    <link name="ur10shoulder_link">
       <visual>
         <geometry>
@@ -101,7 +101,7 @@
       </xacro:cylinder_inertial>
     </link>
-    <joint name="shoulder_lift_joint" type="revolute">
-      <parent link="shoulder_link" />
-      <child link = "upper_arm_link" />
+    <joint name="ur10shoulder_lift_joint" type="revolute">
+      <parent link="ur10shoulder_link" />
+      <child link = "ur10upper_arm_link" />
       <origin xyz="0.0 ${shoulder_offset} 0.0" rpy="0.0 -1.25 0.0" />
       <axis xyz="0 1 0" />
@@ -114,5 +114,5 @@
       <dynamics damping="0.5" friction="10.0"/>
     </joint>
-    <link name="upper_arm_link">
+    <link name="ur10upper_arm_link">
       <visual>
         <geometry>
@@ -129,7 +129,7 @@
       </xacro:cylinder_inertial>
     </link>
-    <joint name="elbow_joint" type="revolute">
-      <parent link="upper_arm_link" />
-      <child link = "forearm_link" />
+    <joint name="ur10elbow_joint" type="revolute">
+      <parent link="ur10upper_arm_link" />
+      <child link = "ur10forearm_link" />
       <origin xyz="0.0 ${elbow_offset} ${upper_arm_length}" rpy="0.0 -1.95 0.0" />
       <axis xyz="0 1 0" />
@@ -142,5 +142,5 @@
       <dynamics damping="0.5" friction="10.0"/>
     </joint>
-    <link name="forearm_link">
+    <link name="ur10forearm_link">
       <visual>
          <geometry>
@@ -157,7 +157,7 @@
       </xacro:cylinder_inertial>
     </link>
-    <joint name="wrist_1_joint" type="revolute">
-      <parent link="forearm_link" />
-      <child link = "wrist_1_link" />
+    <joint name="ur10wrist_1_joint" type="revolute">
+      <parent link="ur10forearm_link" />
+      <child link = "ur10wrist_1_link" />
       <origin xyz="0.0 0.0 ${forearm_length}" rpy="0.0 ${pi / 2.0} 0.0" />
       <axis xyz="0 1 0" />
@@ -170,5 +170,5 @@
       <dynamics damping="0.5" friction="10.0"/>
     </joint>
-    <link name="wrist_1_link">
+    <link name="ur10wrist_1_link">
       <visual>
         <geometry>
@@ -185,7 +185,7 @@
       </xacro:cylinder_inertial>
     </link>
-    <joint name="wrist_2_joint" type="revolute">
-      <parent link="wrist_1_link" />
-      <child link = "wrist_2_link" />
+    <joint name="ur10wrist_2_joint" type="revolute">
+      <parent link="ur10wrist_1_link" />
+      <child link = "ur10wrist_2_link" />
       <origin xyz="0.0 ${wrist_1_length} 0.0" rpy="0.0 0.0 0.0" />
       <axis xyz="0 0 1" />
@@ -198,5 +198,5 @@
       <dynamics damping="0.5" friction="10.0"/>
     </joint>
-    <link name="wrist_2_link">
+    <link name="ur10wrist_2_link">
       <visual>
         <geometry>
@@ -213,7 +213,7 @@
       </xacro:cylinder_inertial>
     </link>
-    <joint name="wrist_3_joint" type="revolute">
-      <parent link="wrist_2_link" />
-      <child link = "wrist_3_link" />
+    <joint name="ur10wrist_3_joint" type="revolute">
+      <parent link="ur10wrist_2_link" />
+      <child link = "ur10wrist_3_link" />
       <origin xyz="0.0 0.0 ${wrist_2_length}" rpy="0.0 0.0 0.0" />
       <axis xyz="0 1 0" />
@@ -226,5 +226,5 @@
       <dynamics damping="0.5" friction="10.0"/>
     </joint>
-    <link name="wrist_3_link">
+    <link name="ur10wrist_3_link">
       <visual>
         <geometry>
@@ -241,10 +241,10 @@
       </xacro:cylinder_inertial>
     </link>
-    <joint name="ee_fixed_joint" type="fixed">
-      <parent link="wrist_3_link" />
-      <child link = "ee_link" />
+    <joint name="ur10ee_fixed_joint" type="fixed">
+      <parent link="ur10wrist_3_link" />
+      <child link = "ur10ee_link" />
       <origin xyz="0.0 ${wrist_3_length} 0.0" rpy="0.0 0.0 ${pi/2.0}" />
     </joint>
-    <link name="ee_link">
+    <link name="ur10ee_link">
       <collision>
         <geometry>
@@ -259,70 +259,70 @@
           <parameters>$(find neo_simulation2)/configs/arms/joint_names_ur10_description.yaml  </parameters>
       </hardware>
-    <joint name="shoulder_pan_joint">
-      <command_interface name="position">
-          <param name="min">-3.15</param>
-          <param name="max">3.15</param>
-      </command_interface>
-      <command_interface name="velocity">
-          <param name="min">-3.15</param>
-          <param name="max">3.15</param>
-      </command_interface>
-      <state_interface name="position"/>
-      <state_interface name="velocity"/>
-      <state_interface name="effort"/>
-    </joint>
-    <joint name="shoulder_lift_joint">
-      <command_interface name="position">
-          <param name="min">-3.15</param>
-          <param name="max">3.15</param>
-      </command_interface>
-      <command_interface name="velocity">
-          <param name="min">-3.15</param>
-          <param name="max">3.15</param>
-      </command_interface>
-      <state_interface name="position"/>
-      <state_interface name="velocity"/>
-      <state_interface name="effort"/>
-    </joint>
-    <joint name="elbow_joint">
-      <command_interface name="position">
-          <param name="min">-3.15</param>
-          <param name="max">3.15</param>
-      </command_interface>
-      <command_interface name="velocity">
-          <param name="min">-3.15</param>
-          <param name="max">3.15</param>
-      </command_interface>
-      <state_interface name="position"/>
-      <state_interface name="velocity"/>
-      <state_interface name="effort"/>
-    </joint>
-    <joint name="wrist_1_joint">
-      <command_interface name="position">
-          <param name="min">-3.15</param>
-          <param name="max">3.15</param>
-      </command_interface>
-      <command_interface name="velocity">
-          <param name="min">-3.15</param>
-          <param name="max">3.15</param>
-      </command_interface>
-      <state_interface name="position"/>
-      <state_interface name="velocity"/>
-      <state_interface name="effort"/>
-    </joint>
-    <joint name="wrist_2_joint">
-      <command_interface name="position">
-          <param name="min">-3.15</param>
-          <param name="max">3.15</param>
-      </command_interface>
-      <command_interface name="velocity">
-          <param name="min">-3.15</param>
-          <param name="max">3.15</param>
-      </command_interface>
-      <state_interface name="position"/>
-      <state_interface name="velocity"/>
-      <state_interface name="effort"/>
-    </joint>
-    <joint name="wrist_3_joint">
+    <joint name="ur10shoulder_pan_joint">
+      <command_interface name="position">
+          <param name="min">-3.15</param>
+          <param name="max">3.15</param>
+      </command_interface>
+      <command_interface name="velocity">
+          <param name="min">-3.15</param>
+          <param name="max">3.15</param>
+      </command_interface>
+      <state_interface name="position"/>
+      <state_interface name="velocity"/>
+      <state_interface name="effort"/>
+    </joint>
+    <joint name="ur10shoulder_lift_joint">
+      <command_interface name="position">
+          <param name="min">-3.15</param>
+          <param name="max">3.15</param>
+      </command_interface>
+      <command_interface name="velocity">
+          <param name="min">-3.15</param>
+          <param name="max">3.15</param>
+      </command_interface>
+      <state_interface name="position"/>
+      <state_interface name="velocity"/>
+      <state_interface name="effort"/>
+    </joint>
+    <joint name="ur10elbow_joint">
+      <command_interface name="position">
+          <param name="min">-3.15</param>
+          <param name="max">3.15</param>
+      </command_interface>
+      <command_interface name="velocity">
+          <param name="min">-3.15</param>
+          <param name="max">3.15</param>
+      </command_interface>
+      <state_interface name="position"/>
+      <state_interface name="velocity"/>
+      <state_interface name="effort"/>
+    </joint>
+    <joint name="ur10wrist_1_joint">
+      <command_interface name="position">
+          <param name="min">-3.15</param>
+          <param name="max">3.15</param>
+      </command_interface>
+      <command_interface name="velocity">
+          <param name="min">-3.15</param>
+          <param name="max">3.15</param>
+      </command_interface>
+      <state_interface name="position"/>
+      <state_interface name="velocity"/>
+      <state_interface name="effort"/>
+    </joint>
+    <joint name="ur10wrist_2_joint">
+      <command_interface name="position">
+          <param name="min">-3.15</param>
+          <param name="max">3.15</param>
+      </command_interface>
+      <command_interface name="velocity">
+          <param name="min">-3.15</param>
+          <param name="max">3.15</param>
+      </command_interface>
+      <state_interface name="position"/>
+      <state_interface name="velocity"/>
+      <state_interface name="effort"/>
+    </joint>
+    <joint name="ur10wrist_3_joint">
       <command_interface name="position">
           <param name="min">-3.15</param>
