Commit message: Adding Robotiq gripper to ur10 arm (#105)
* Switched base_link and base_footprint to follow Nav2 convention

* Added launch argument to include docking adapter(True for MPO-700 only)

* Updated mp_500 and mp_400 urdf

* Updated the odometry_frame param in planar move controller

* Attatched Robotiq 2f 140 gripper to the arm and created the necessary launch file to visualize the robot and control the joints using joint state publisher gui

File: components/common_macro/gazebo_object_controller_macro.xacro (robot description, xacro)
@@ -23,6 +23,6 @@
                 <publish_odom_tf>true</publish_odom_tf>
                 <!-- Frame IDs -->
-                <odometryFrame>${odom_frame}</odometryFrame>
-                <robotBaseFrame>${base_frame}</robotBaseFrame>
+                <odometry_frame>${odom_frame}</odometry_frame>
+                <robot_base_frame>${base_frame}</robot_base_frame>
                 <!-- Set odom covariance -->
                 <covariance_x>0.0001</covariance_x>

File: robots/mpo_700/urdf/mpo_700_body.urdf.xacro (robot description, xacro)
@@ -2,12 +2,4 @@
 <robot xmlns:xacro="http://www.ros.org/wiki/xacro" name="mpo_700">
     <link name="base_footprint"/>
-    <joint name="base_footprint_joint" type="fixed">
-        <origin rpy="0 0 0" xyz="0 0 0"/>
-        <axis xyz="0 0 -1"/>
-        <!-- <limit effort="1000.0" lower="-1e+16" upper="1e+16" velocity="15"/> -->
-        <joint_properties damping="1" friction="1"/>
-        <parent link="base_footprint"/>
-        <child link="base_link"/>
-    </joint>
     <link name="base_link">
         <inertial>
@@ -29,4 +21,12 @@
         </collision>
     </link>
+    <joint name="base_footprint_joint" type="fixed">
+        <origin rpy="0 0 0" xyz="0 0 0"/>
+        <axis xyz="0 0 -1"/>
+        <!-- <limit effort="1000.0" lower="-1e+16" upper="1e+16" velocity="15"/> -->
+        <joint_properties damping="1" friction="1"/>
+        <parent link="base_link"/>
+        <child link="base_footprint"/>
+    </joint>
     <!-- Sensors -->
     <joint name="lidar_1_joint" type="fixed">
@@ -170,7 +170,9 @@
     </xacro:mpo_700_wheel>
     <!-- Import docking adapter -->
-    <xacro:include filename="$(find neo_simulation2)/robots/mpo_700/urdf/macro/docking_adapter.xacro"/>
-    <xacro:docking_adapter name="docking_adapter" parent="base_link">
-        <origin xyz="-0.300 0 0.320" rpy="0 0 -1.57" />
-    </xacro:docking_adapter>
+    <xacro:if value="$(arg use_docking_adapter)">
+        <xacro:include filename="$(find neo_simulation2)/robots/mpo_700/urdf/macro/docking_adapter.xacro"/>
+        <xacro:docking_adapter name="docking_adapter" parent="base_link">
+            <origin xyz="-0.300 0 0.320" rpy="0 0 -1.57" />
+        </xacro:docking_adapter>
+    </xacro:if>
 </robot>

Commit message: Revert "Adding Robotiq gripper to ur10 arm (#105)"
This reverts commit 3dd49485a9abfd2d1f87da0e9a5ecfe02a707d04.

File: components/common_macro/gazebo_object_controller_macro.xacro (robot description, xacro)
@@ -23,6 +23,6 @@
                 <publish_odom_tf>true</publish_odom_tf>
                 <!-- Frame IDs -->
-                <odometry_frame>${odom_frame}</odometry_frame>
-                <robot_base_frame>${base_frame}</robot_base_frame>
+                <odometryFrame>${odom_frame}</odometryFrame>
+                <robotBaseFrame>${base_frame}</robotBaseFrame>
                 <!-- Set odom covariance -->
                 <covariance_x>0.0001</covariance_x>

File: robots/mp_400/urdf/mp_400_body.urdf.xacro (robot description, xacro)
@@ -2,4 +2,12 @@
 <robot xmlns:xacro="http://www.ros.org/wiki/xacro" name="mp_400">
     <link name="base_footprint"/>
+    <joint name="base_footprint_joint" type="fixed">
+        <origin rpy="0 0 0" xyz="0 0 0"/>
+        <axis xyz="0 0 -1"/>
+        <!-- <limit effort="1000.0" lower="-1e+16" upper="1e+16" velocity="3.5"/> -->
+        <joint_properties damping="1" friction="1"/>
+        <parent link="base_footprint"/>
+        <child link="base_link"/>
+    </joint>
     <link name="base_link">
         <inertial>
@@ -21,12 +29,4 @@
         </collision>
     </link>
-    <joint name="base_footprint_joint" type="fixed">
-        <origin rpy="0 0 0" xyz="0 0 0"/>
-        <axis xyz="0 0 -1"/>
-        <!-- <limit effort="1000.0" lower="-1e+16" upper="1e+16" velocity="3.5"/> -->
-        <joint_properties damping="1" friction="1"/>
-        <parent link="base_link"/>
-        <child link="base_footprint"/>
-    </joint>
     <!-- Sensors -->
     <joint name="lidar_1_joint" type="fixed">

File: robots/mp_400/urdf/mp_400_gazebo.urdf.xacro (robot description, xacro)
@@ -27,5 +27,5 @@
         odometry_topic="odom"
         odom_frame="odom"
-        base_frame="base_link"
+        base_frame="base_footprint"
         max_wheel_torque="1000"
         max_acceleration="20.0"

File: robots/mp_500/urdf/mp_500_body.urdf.xacro (robot description, xacro)
@@ -2,4 +2,12 @@
 <robot xmlns:xacro="http://www.ros.org/wiki/xacro" name="mp_500">
     <link name="base_footprint"/>
+    <joint name="base_footprint_joint" type="fixed">
+        <origin rpy="0 0 0" xyz="0 0 0"/>
+        <axis xyz="0 0 -1"/>
+        <!-- <limit effort="1000.0" lower="-1e+16" upper="1e+16" velocity="3.5"/> -->
+        <joint_properties damping="1" friction="1"/>
+        <parent link="base_footprint"/>
+        <child link="base_link"/>
+    </joint>
     <link name="base_link">
         <inertial>
@@ -21,12 +29,4 @@
         </collision>
     </link>
-    <joint name="base_footprint_joint" type="fixed">
-        <origin rpy="0 0 0" xyz="0 0 0"/>
-        <axis xyz="0 0 -1"/>
-        <!-- <limit effort="1000.0" lower="-1e+16" upper="1e+16" velocity="3.5"/> -->
-        <joint_properties damping="1" friction="1"/>
-        <parent link="base_link"/>
-        <child link="base_footprint"/>
-    </joint>
     <joint name="caster_wheel_joint" type="fixed">
         <origin rpy="-1.570796 0 1.570796 " xyz="-0.43 0. 0.176"/>

File: robots/mp_500/urdf/mp_500_gazebo.urdf.xacro (robot description, xacro)
@@ -17,5 +17,5 @@
         odometry_topic="odom"
         odom_frame="odom"
-        base_frame="base_link"
+        base_frame="base_footprint"
         max_wheel_torque="200"
         max_acceleration="1.0"

File: robots/mpo_500/urdf/mpo_500_body.urdf.xacro (robot description, xacro)
@@ -2,4 +2,12 @@
 <robot xmlns:xacro="http://www.ros.org/wiki/xacro" name="mpo_500">
     <link name="base_footprint"/>
+    <joint name="base_footprint_joint" type="fixed">
+        <origin rpy="0 0 0" xyz="0 0 0"/>
+        <axis xyz="0 0 -1"/>
+        <!-- <limit effort="1000.0" lower="-1e+16" upper="1e+16" velocity="15"/> -->
+        <joint_properties damping="1" friction="1"/>
+        <parent link="base_footprint"/>
+        <child link="base_link"/>
+    </joint>
     <link name="base_link">
         <inertial>
@@ -21,12 +29,4 @@
         </collision>
     </link>
-    <joint name="base_footprint_joint" type="fixed">
-        <origin rpy="0 0 0" xyz="0 0 0"/>
-        <axis xyz="0 0 -1"/>
-        <!-- <limit effort="1000.0" lower="-1e+16" upper="1e+16" velocity="15"/> -->
-        <joint_properties damping="1" friction="1"/>
-        <parent link="base_link"/>
-        <child link="base_footprint"/>
-    </joint>
     <!-- Sensors -->
     <joint name="lidar_1_joint" type="fixed">

File: robots/mpo_700/mpo_700.urdf.xacro (robot description, xacro)
@@ -4,6 +4,4 @@
     <!--set use_gazebo = false for implementation on real robot-->
     <xacro:arg name="use_gazebo" default="true"/>
-    <!--set use_docking_adapter = true to use adapter with the robot-->
-    <xacro:arg name="use_docking_adapter" default="false"/>
     <!--set arm name to include the arm in the simulation-->
     <xacro:arg name="arm_type" default=""/>

File: robots/mpo_700/urdf/mpo_700_body.urdf.xacro (robot description, xacro)
@@ -2,4 +2,12 @@
 <robot xmlns:xacro="http://www.ros.org/wiki/xacro" name="mpo_700">
     <link name="base_footprint"/>
+    <joint name="base_footprint_joint" type="fixed">
+        <origin rpy="0 0 0" xyz="0 0 0"/>
+        <axis xyz="0 0 -1"/>
+        <!-- <limit effort="1000.0" lower="-1e+16" upper="1e+16" velocity="15"/> -->
+        <joint_properties damping="1" friction="1"/>
+        <parent link="base_footprint"/>
+        <child link="base_link"/>
+    </joint>
     <link name="base_link">
         <inertial>
@@ -21,12 +29,4 @@
         </collision>
     </link>
-    <joint name="base_footprint_joint" type="fixed">
-        <origin rpy="0 0 0" xyz="0 0 0"/>
-        <axis xyz="0 0 -1"/>
-        <!-- <limit effort="1000.0" lower="-1e+16" upper="1e+16" velocity="15"/> -->
-        <joint_properties damping="1" friction="1"/>
-        <parent link="base_link"/>
-        <child link="base_footprint"/>
-    </joint>
     <!-- Sensors -->
     <joint name="lidar_1_joint" type="fixed">
@@ -170,9 +170,7 @@
     </xacro:mpo_700_wheel>
     <!-- Import docking adapter -->
-    <xacro:if value="$(arg use_docking_adapter)">
-        <xacro:include filename="$(find neo_simulation2)/robots/mpo_700/urdf/macro/docking_adapter.xacro"/>
-        <xacro:docking_adapter name="docking_adapter" parent="base_link">
-            <origin xyz="-0.300 0 0.320" rpy="0 0 -1.57" />
-        </xacro:docking_adapter>
-    </xacro:if>
+    <xacro:include filename="$(find neo_simulation2)/robots/mpo_700/urdf/macro/docking_adapter.xacro"/>
+    <xacro:docking_adapter name="docking_adapter" parent="base_link">
+        <origin xyz="-0.300 0 0.320" rpy="0 0 -1.57" />
+    </xacro:docking_adapter>
 </robot>

File: robots/mpo_700/urdf/mpo_700_gazebo.urdf.xacro (robot description, xacro)
@@ -15,5 +15,5 @@
         controller_update_rate="${controller_update_rate}"
         odom_frame="odom"
-        base_frame="base_link"
+        base_frame="base_footprint"
         covariance_yaw="0.0001"
     />
